Commit message: add new map + add GPS

File: urdf/bcr_bot.xacro (robot description, xacro)
@@ -241,4 +241,29 @@
         </joint>
     </xacro:if>
-    <!-- ............................................................................... -->
+<!-- ............................. GPS ........................................ -->
+    <link name="gps_link">
+        <visual>
+            <origin xyz="0 0 0" rpy="0 0 0" />
+            <geometry>
+                <box size="0.05 0.05 0.02"/>
+            </geometry>
+            <material name="black"/>
+        </visual>
+        <collision>
+            <origin xyz="0 0 0" rpy="0 0 0" />
+            <geometry>
+                <box size="0.05 0.05 0.02"/>
+            </geometry>
+        </collision>
+        <inertial>
+            <mass value="0.05"/>
+            <xacro:box_inertia m="0.05" x="0.05" y="0.05" z="0.02"/>
+        </inertial>
+    </link>
+    <joint name="gps_joint" type="fixed">
+        <parent link="roof_link"/>
+        <child link="gps_link"/>
+        <origin xyz="0.0 0.0 0.02" rpy="0.0 0.0 0.0"/>
+    </joint>
+        <!-- ............................................................................... -->
 </robot>

File: urdf/gz.xacro (robot description, xacro)
@@ -7,4 +7,6 @@
         </plugin>
         <plugin filename="gz-sim-imu-system" name="gz::sim::systems::Imu">
+        </plugin>
+        <plugin filename="gz-sim-navsat-system" name="gz::sim::systems::NavSat">
         </plugin>
         <plugin filename="gz-sim-joint-state-publisher-system" name="gz::sim::systems::JointStatePublisher">
@@ -105,4 +107,13 @@
         </sensor>
     </gazebo>
+    <!-- ........................... GPS config ................................... -->
+    <gazebo reference="gps_link">
+        <sensor name="navsat_sensor" type="navsat">
+            <always_on>1</always_on>
+            <update_rate>10.0</update_rate>
+            <gz_frame_id>gps_link</gz_frame_id>
+            <topic>gps/fix</topic>
+        </sensor>
+    </gazebo>
     <!-- ........................... Stereo camera ................................... -->
     <xacro:if value="$(arg stereo_camera_enabled)">
